Commit message: Create gazebo controllers and sim

File: abb_irb2600_support/urdf/irb2600_12_165_macro.xacro (robot description, xacro)
@@ -4,4 +4,6 @@
   <xacro:macro name="abb_irb2600_12_165" params="prefix">
     <!-- links -->
+     <link name="zero_link">
+     </link>
     <link name="${prefix}base_link">
       <visual>
@@ -18,4 +20,11 @@
         </geometry>
       </collision>
+      <inertial>
+        <origin xyz="0 0 0" rpy="0 0 0"/>
+        <mass value="100.0"/> <!-- in kg -->
+        <inertia ixx="0.8" ixy="0.0" ixz="0.0"
+                iyy="0.8" iyz="0.0"
+                izz="0.8"/>
+      </inertial>
     </link>
     <link name="${prefix}link_1">
@@ -33,4 +42,11 @@
         </geometry>
       </collision>
+      <inertial>
+        <origin xyz="0 0 0" rpy="0 0 0"/>
+        <mass value="25.0"/> <!-- in kg -->
+        <inertia ixx="0.3" ixy="0.0" ixz="0.0"
+                iyy="0.3" iyz="0.0"
+                izz="0.3"/>
+      </inertial>
     </link>
     <link name="${prefix}link_2">
@@ -48,4 +64,11 @@
         </geometry>
       </collision>
+      <inertial>
+        <origin xyz="0 0 0" rpy="0 0 0"/>
+        <mass value="25.0"/> <!-- in kg -->
+        <inertia ixx="0.3" ixy="0.0" ixz="0.0"
+                iyy="0.3" iyz="0.0"
+                izz="0.3"/>
+      </inertial>
     </link>
     <link name="${prefix}link_3">
@@ -63,4 +86,11 @@
         </geometry>
       </collision>
+      <inertial>
+        <origin xyz="0 0 0" rpy="0 0 0"/>
+        <mass value="15.0"/> <!-- in kg -->
+        <inertia ixx="0.2" ixy="0.0" ixz="0.0"
+                iyy="0.2" iyz="0.0"
+                izz="0.2"/>
+      </inertial>
     </link>
     <link name="${prefix}link_4">
@@ -78,4 +108,11 @@
         </geometry>
       </collision>
+      <inertial>
+        <origin xyz="0 0 0" rpy="0 0 0"/>
+        <mass value="25.0"/> <!-- in kg -->
+        <inertia ixx="0.3" ixy="0.0" ixz="0.0"
+                iyy="0.3" iyz="0.0"
+                izz="0.3"/>
+      </inertial>
     </link>
     <link name="${prefix}link_5">
@@ -93,4 +130,11 @@
         </geometry>
       </collision>
+      <inertial>
+        <origin xyz="0 0 0" rpy="0 0 0"/>
+        <mass value="15.0"/> <!-- in kg -->
+        <inertia ixx="0.2" ixy="0.0" ixz="0.0"
+                iyy="0.2" iyz="0.0"
+                izz="0.2"/>
+      </inertial>
     </link>
     <link name="${prefix}link_6">
@@ -98,5 +142,5 @@
         <origin xyz="0 0 0" rpy="0 0 0" />
         <geometry>
-          <mesh filename="package://abb_irb2600_support/meshes/irb2600_12_165/visual/link_6.stl" />
+          <mesh filename="package://abb_irb2600_support/meshes/irb2600_12_165/visual/link_6.stl" scale="0.1 0.1 0.1"/>
         </geometry>
         <material name="">
@@ -107,9 +151,21 @@
         <origin xyz="0 0 0" rpy="0 0 0" />
         <geometry>
-          <mesh filename="package://abb_irb2600_support/meshes/irb2600_12_165/collision/link_6.stl" />
-        </geometry>
-      </collision>
+          <mesh filename="package://abb_irb2600_support/meshes/irb2600_12_165/collision/link_6.stl" scale="0.1 0.1 0.1"/>
+        </geometry>
+      </collision>
+      <inertial>
+        <origin xyz="0 0 0" rpy="0 0 0"/>
+        <mass value="5.0"/> <!-- in kg -->
+        <inertia ixx="0.1" ixy="0.0" ixz="0.0"
+                iyy="0.1" iyz="0.0"
+                izz="0.1"/>
+      </inertial>
     </link>
     <!-- Joints -->
+     <joint name="zero_joint" type="fixed">
+       <origin xyz="0 0 0" rpy="0 0 0"/>
+       <parent link="zero_link"/>
+       <child link="${prefix}base_link"/>
+     </joint>
     <joint name="${prefix}joint_1" type="revolute">
       <origin xyz="0 0 0.445" rpy="0 0 0" />
@@ -175,4 +231,69 @@
       <child link="${prefix}tool0" />
     </joint>
+    <transmission name="${prefix}tran_1">
+      <type>transmission_interface/SimpleTransmission</type>
+      <joint name="${prefix}joint_1">
+        <hardwareInterface>hardware_interface/PositionJointInterface</hardwareInterface>
+      </joint>
+      <actuator name="${prefix}motor_1">
+        <hardwareInterface>hardware_interface/PositionJointInterface</hardwareInterface>
+        <mechanicalReduction>1</mechanicalReduction>
+      </actuator>
+    </transmission>
+    <transmission name="${prefix}tran_2">
+      <type>transmission_interface/SimpleTransmission</type>
+      <joint name="${prefix}joint_2">
+        <hardwareInterface>hardware_interface/PositionJointInterface</hardwareInterface>
+      </joint>
+      <actuator name="${prefix}motor_2">
+        <hardwareInterface>hardware_interface/PositionJointInterface</hardwareInterface>
+        <mechanicalReduction>1</mechanicalReduction>
+      </actuator>
+    </transmission>
+    <transmission name="${prefix}tran_3">
+      <type>transmission_interface/SimpleTransmission</type>
+      <joint name="${prefix}joint_3">
+        <hardwareInterface>hardware_interface/PositionJointInterface</hardwareInterface>
+      </joint>
+      <actuator name="${prefix}motor_3">
+        <hardwareInterface>hardware_interface/PositionJointInterface</hardwareInterface>
+        <mechanicalReduction>1</mechanicalReduction>
+      </actuator>
+    </transmission>
+    <transmission name="${prefix}tran_4">
+      <type>transmission_interface/SimpleTransmission</type>
+      <joint name="${prefix}joint_4">
+        <hardwareInterface>hardware_interface/PositionJointInterface</hardwareInterface>
+      </joint>
+      <actuator name="${prefix}motor_4">
+        <hardwareInterface>hardware_interface/PositionJointInterface</hardwareInterface>
+        <mechanicalReduction>1</mechanicalReduction>
+      </actuator>
+    </transmission>
+    <transmission name="${prefix}tran_5">
+      <type>transmission_interface/SimpleTransmission</type>
+      <joint name="${prefix}joint_5">
+        <hardwareInterface>hardware_interface/PositionJointInterface</hardwareInterface>
+      </joint>
+      <actuator name="${prefix}motor_5">
+        <hardwareInterface>hardware_interface/PositionJointInterface</hardwareInterface>
+        <mechanicalReduction>1</mechanicalReduction>
+      </actuator>
+    </transmission>
+    <transmission name="${prefix}tran_6">
+      <type>transmission_interface/SimpleTransmission</type>
+      <joint name="${prefix}joint_6">
+        <hardwareInterface>hardware_interface/PositionJointInterface</hardwareInterface>
+      </joint>
+      <actuator name="${prefix}motor_6">
+        <hardwareInterface>hardware_interface/PositionJointInterface</hardwareInterface>
+        <mechanicalReduction>1</mechanicalReduction>
+      </actuator>
+    </transmission>
+  <gazebo>
+    <plugin name="gazebo_ros_control" filename="libgazebo_ros_control.so">
+      <robotNamespace>/</robotNamespace>
+    </plugin>
+  </gazebo>
   </xacro:macro>
 </robot>
